File: KiCad/slime_tracker.kicad_sch (KiCad schematic)
At the start: 64 parts, among them J1 batt, J2 Extension, J3 USB_C_Receptacle_PowerOnly_6P, SW1 SW_DPDT_x2, U1 TP4056, U3 TPS7A0333PDBVR, U4 ESP32 SUPER MINI C3, U5 TPS61090

Commit message: rev03 almost
com
Parts:
- removed H1, H2: MountingHole, MountingHole:MountingHole_3.2mm_M3, symbol Mechanical:MountingHole
- C5: footprint Capacitor_SMD:C_0603_1608Metric -> Capacitor_SMD:C_0805_2012Metric
Other:
- note added: "SOD-123"
- note removed: "SOD-323 B5819W"
Changed lines of the file:
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@@
 		)
 	)
-	(text "CAP SIZE 0603\n\n"
+	(text "CAP SIZE 0805\n\n\n"
 		(exclude_from_sim no)
-		(at 116.332 43.434 0)
+		(at 116.332 44.196 0)
 		(effects
 			(font
@@
 		)
 	)
-	(text "CAP SIZE 0603\n\n"
+	(text "CAP SIZE 0805\n\n\n"
 		(exclude_from_sim no)
 		(at 106.426 146.812 0)
@@
 		)
 	)
-	(text "SOD-323\n\nB5819W \n"
+	(text "SOD-123\n"
 		(exclude_from_sim no)
-		(at 236.22 166.116 0)
+		(at 240.538 165.608 0)
 		(effects
 			(font
@@
 			)
 		)
-		(property "Footprint" "Capacitor_SMD:C_0603_1608Metric"
+		(property "Footprint" "Capacitor_SMD:C_0805_2012Metric"
 			(at 114.6048 33.02 0)
 			(effects
@@
 	)
 	(symbol
-		(lib_id "Mechanical:MountingHole")
-		(at 414.02 20.32 0)
-		(unit 1)
-		(exclude_from_sim no)
-		(in_bom no)
-		(on_board yes)
-		(dnp no)
-		(property "Reference" "H2"
-			(at 416.56 19.0499 0)
-			(effects
-				(font
-					(size 1.27 1.27)
-				)
-				(justify left)
-			)
-		)
-		(property "Value" "MountingHole"
-			(at 416.56 21.5899 0)
-			(effects
-				(font
-					(size 1.27 1.27)
-				)
-				(justify left)
-			)
-		)
-		(property "Footprint" "MountingHole:MountingHole_3.2mm_M3"
-			(at 414.02 20.32 0)
-			(effects
-				(font
-					(size 1.27 1.27)
-				)
-				(hide yes)
-			)
-		)
-		(property "Datasheet" "~"
-			(at 414.02 20.32 0)
-			(effects
-				(font
-					(size 1.27 1.27)
-				)
-				(hide yes)
-			)
-		)
-		(property "Description" "Mounting Hole without connection"
-			(at 414.02 20.32 0)
-			(effects
-				(font
-					(size 1.27 1.27)
-				)
-				(hide yes)
-			)
-		)
-		(instances
-			(project ""
-				(path "/9f3f9b38-d2e1-497f-9960-ea0c5443957e"
-					(reference "H2")
-					(unit 1)
-				)
-			)
-		)
-	)
-	(symbol
 		(lib_id "power:GNDREF")
 		(at 326.39 128.27 0)
@@
 					(unit 1)
 				)
-			)
-		)
-	)
-	(symbol
-		(lib_id "Mechanical:MountingHole")
-		(at 414.02 13.97 0)
-		(unit 1)
-		(exclude_from_sim no)
-		(in_bom no)
-		(on_board yes)
-		(dnp no)
-		(property "Reference" "H1"
-			(at 416.56 12.6999 0)
-			(effects
-				(font
-					(size 1.27 1.27)
-				)
-				(justify left)
-			)
-		)
-		(property "Value" "MountingHole"
-			(at 416.56 15.2399 0)
-			(effects
-				(font
-					(size 1.27 1.27)
-				)
-				(justify left)
-			)
-		)
-		(property "Footprint" "MountingHole:MountingHole_3.2mm_M3"
-			(at 414.02 13.97 0)
-			(effects
-				(font
-					(size 1.27 1.27)
-				)
-				(hide yes)
-			)
-		)
-		(property "Datasheet" "~"
-			(at 414.02 13.97 0)
-			(effects
-				(font
-					(size 1.27 1.27)
-				)
-				(hide yes)
-			)
-		)
-		(property "Description" "Mounting Hole without connection"
-			(at 414.02 13.97 0)
-			(effects
-				(font
-					(size 1.27 1.27)
-				)
-				(hide yes)
-			)
-		)
-		(instances
-			(project ""
-				(path "/9f3f9b38-d2e1-497f-9960-ea0c5443957e"
-					(reference "H1")
-					(unit 1)
-				)
