File: KiCad/slime_tracker.kicad_pcb (KiCad board)
At the start: 2 copper layers, 80.2 x 32 mm, 64 parts, among them J1 batt, J2 Extension, J3 USB_C_Receptacle_PowerOnly_6P, SW1 SW_DPDT_x2, U1 TP4056, U3 TPS7A0333PDBVR, U4 ESP32 SUPER MINI C3, U5 TPS61090

Commit message: board cut
cc
Parts:
- removed H1, H2: MountingHole, MountingHole:MountingHole_3.2mm_M3
- moved H6 5.99 mm to (156.9, 41.5)
- moved H5 0.71 mm to (95.6, 38.3)
- moved SW1 0.35 mm to (88.1, 40.8)
Routing:
- net BAT-_TO_BOOST: track 24.7 -> 25.7 mm
- net BAT-: vias 132 -> 166
Other:
- board size 80.2 x 32 mm -> 80.4 x 32 mm
